Commit message: feat: real link dimensions and mesh files from HexapodV2.step CAD
Replaced all placeholder dimensions in common.xacro with measurements taken
directly from HexapodV2.step (the actual CAD assembly) on 2026-08-29:

  coxa_length  0.045 -> 0.0764 m
  femur_length 0.075 -> 0.0859 m
  tibia_length 0.130 -> 0.1194 m
  coxa_tilt_deg   55 -> 50 deg
  leg_splay_deg   40 -> 40 (confirmed against the body's own mount sketch)
  body_length/width  0.200x0.120 -> 0.300x0.223 m
  body_mount_x/y     0.080/0.060 -> 0.1383/0.0663 m

Link lengths came from the distance between servo-shaft bore centers at
each joint (body-coxa, coxa-femur, femur-tibia), found by matching aligned
mounting-hole patterns between adjacent CAD solids and cross-validated
against a a manual measurement in Fusion. tibia_length is to the farthest
point on the tibia body from its joint. coxa_tilt_deg is the femur's real
droop below horizontal; the coxa's own smaller built-in droop (~25 deg) is
intentionally folded into that single value rather than modeled as a
second tilt stage, keeping the existing 3-DOF architecture and
leg_kinematics.py's planar-arm IK reduction unchanged.

Synced hexapod_control/config/gait.yaml and leg_kinematics.py's
LegGeometry defaults to match, per common.xacro's own "propagate from
here" note. Existing gait.yaml stance/step parameters were checked against
the new (slightly larger) reachable envelope and still fit safely.

Also added the four real mesh files (body/coxa/femur/tibia.stl), generated
programmatically from the same STEP file's solids: each repositioned so
its local origin sits exactly at its proximal joint with the link's long
axis along +X, matching leg.xacro's mesh convention exactly (self-
consistency check: the repositioned tibia's farthest point lands at
x=119.4mm, exactly tibia_length). Exported at a coarser tessellation
tolerance than CAD-native to keep triangle counts reasonable (~3000/leg
part, ~9000 for the body) since Gazebo has to load 18 leg meshes; CAD-
defeaturing the screw holes was tried but didn't meaningfully help, the
triangle cost is mostly in fillets/curves rather than the holes.

use_meshes now defaults to true in hexapod.urdf.xacro.

Verified: FK/IK round-trip test still passes with the new geometry, xacro
still processes cleanly with use_meshes on, and a full Gazebo sim launch
still reaches both controllers active (takes ~30-35s to load now instead
of ~20s, real meshes vs primitive boxes).

Co-Authored-By: Claude Sonnet 5 <noreply@anthropic.com>

File: hexapod_description/urdf/common.xacro (robot description, xacro)
@@ -13,32 +13,46 @@
 <robot xmlns:xacro="http://www.ros.org/wiki/xacro">
   <!-- ========== body ========== -->
-  <xacro:property name="body_length"    value="0.200"/>
-  <xacro:property name="body_width"     value="0.120"/>
+  <!-- Measured 2026-08-29 from HexapodV2.step (bounding box of HexapodMainBody). -->
+  <xacro:property name="body_length"    value="0.300"/>
+  <xacro:property name="body_width"     value="0.223"/>
   <xacro:property name="body_thickness" value="0.040"/>
   <xacro:property name="body_mass"      value="1.50"/>
-  <!-- Ride height: ground to base_link origin. -->
-  <xacro:property name="body_height"    value="0.120"/>
-  <!-- Coxa joint positions on the body. -->
-  <xacro:property name="body_mount_x" value="0.080"/>
-  <xacro:property name="body_mount_y" value="0.060"/>
+  <!-- Ride height: ground to base_link origin. Not a direct CAD measurement -
+       tune alongside gait.yaml's stance_drop once the gait is walking. -->
+  <xacro:property name="body_height"    value="0.135"/>
+  <!-- Coxa joint positions on the body. Measured from the body-coxa joint's
+       servo-shaft bore in the CAD assembly (see common.xacro's HARDWARE
+       VALUES note - re-measure there first if this changes). -->
+  <xacro:property name="body_mount_x" value="0.1383"/>
+  <xacro:property name="body_mount_y" value="0.0663"/>
   <!-- Leg splay: how far the front/rear legs point off the forward centreline,
        viewed from above. Mid legs are always 90 deg (straight out sideways).
-       40 deg matches the mount geometry: atan2(0.060, 0.080) = 36.9 deg, so the
-       legs point very nearly radially outward from the body corners. -->
+       Confirmed directly from the body's own mounting-pattern sketch in CAD
+       (measured 140 deg between the forward axis and a rear mount line, i.e.
+       180 - 40). -->
   <xacro:property name="leg_splay_deg" value="40"/>
-  <!-- ========== leg segments ========== -->
-  <xacro:property name="coxa_length"  value="0.045"/>
-  <xacro:property name="femur_length" value="0.075"/>
-  <xacro:property name="tibia_length" value="0.130"/>
-  <!-- THE 55 DEGREE TILT.
-       The femur joint's mounting frame is pitched 55 deg downward relative to
-       the coxa, so with all joints at zero the leg already slopes toward the
+  <!-- ========== leg segments ==========
+       Measured 2026-08-29 from HexapodV2.step: distance between the servo-
+       shaft bore centres at each joint (body-coxa, coxa-femur, femur-tibia),
+       tibia_length to the farthest point on the tibia body from its joint. -->
+  <xacro:property name="coxa_length"  value="0.0764"/>
+  <xacro:property name="femur_length" value="0.0859"/>
+  <xacro:property name="tibia_length" value="0.1194"/>
+  <!-- THE COXA TILT.
+       The femur joint's mounting frame is pitched downward relative to the
+       coxa, so with all joints at zero the leg already slopes toward the
        ground instead of sticking straight out. This is a fixed mechanical
-       offset in the bracket, NOT a commandable joint.
+       offset in the bracket, NOT a commandable joint. Measured as the real
+       femur droop below horizontal at the CAD's rest pose - the coxa itself
+       also has a smaller built-in droop (~25 deg) that this model doesn't
+       represent separately; folding it into a single tilt at the femur is a
+       deliberate simplification (matches the existing 3-DOF architecture and
+       leg_kinematics.py's planar-arm reduction) rather than adding a second
+       fixed tilt stage.
        Consequence for the IK: the femur command angle is measured FROM this
        tilted frame, so the femur's true angle below horizontal is
-       (55 deg + femur_command). hexapod_control accounts for this - see
-       leg_kinematics.py. -->
-  <xacro:property name="coxa_tilt_deg" value="55"/>
+       (coxa_tilt_deg + femur_command). hexapod_control accounts for this -
+       see leg_kinematics.py. -->
+  <xacro:property name="coxa_tilt_deg" value="50"/>
   <xacro:property name="coxa_mass"  value="0.08"/>
   <xacro:property name="femur_mass" value="0.12"/>

File: hexapod_description/urdf/hexapod.urdf.xacro (robot description, xacro)
@@ -14,6 +14,7 @@
        gz_ros2_control plugin can find it at spawn time. -->
   <xacro:arg name="controllers_file" default=""/>
-  <!-- Flip to true once real meshes land in hexapod_description/meshes. -->
-  <xacro:arg name="use_meshes" default="false"/>
+  <!-- Real meshes landed 2026-08-29 (exported from HexapodV2.step) - on by
+       default now. Set false for the primitive-box fallback. -->
+  <xacro:arg name="use_meshes" default="true"/>
   <!-- Set false for a plain URDF with no Gazebo / ros2_control tags. -->
   <xacro:arg name="simulation" default="true"/>

Commit message: fix: mesh orientation didn't match the kinematic chain, and add missing servos
Two things, both surfaced by actually looking at the rendered robot:

1. Each leg segment's mesh was aligned to its OWN real-world CAD direction
   independently (coxa to its real ~25deg droop, femur to its own real
   direction, etc). But the kinematic model deliberately treats the coxa
   as perfectly level (coxa_joint is pure yaw, zero pitch - all droop is
   folded into a single fixed tilt at the femur, a documented
   simplification). A mesh built from the real tilted vector can never
   match that - the coxa_joint has no way to pitch it back level - so it
   visually drooped no matter what, and every downstream mesh (each
   aligned to its own noisy real direction) compounded the mismatch into
   a visibly disconnected, scattered leg.

   Fixed by reconstructing each segment's direction from the model's own
   convention instead of raw CAD vectors: coxa horizontal (using only the
   horizontal projection of the real coxa vector), femur pitched down
   exactly coxa_tilt_deg from coxa's heading, tibia continuing in that
   same straight line (a zero tibia command means no additional bend).
   This also meant coxa_length needed to become the horizontal-only
   projection (69.5mm) instead of the real 3D distance (76.4mm) - using
   the 3D distance overstated how far the (actually-level) modeled coxa
   reaches out.

2. The servo motors were missing entirely - only used the 3 large bracket
   solids per leg, none of the repeated hardware solids. Since each link
   physically carries the servo that drives the NEXT joint, merged: body
   + coxa's own driving servo, coxa bracket + femur's driving servo, femur
   bracket + tibia's driving servo, tibia bracket alone (nothing rotates
   after it, no servo to carry). Identified which hardware solid belongs
   to which link by proximity to each bracket's own bounding box.

Co-Authored-By: Claude Sonnet 5 <noreply@anthropic.com>

File: hexapod_description/urdf/common.xacro (robot description, xacro)
@@ -35,6 +35,16 @@
        Measured 2026-08-29 from HexapodV2.step: distance between the servo-
        shaft bore centres at each joint (body-coxa, coxa-femur, femur-tibia),
-       tibia_length to the farthest point on the tibia body from its joint. -->
-  <xacro:property name="coxa_length"  value="0.0764"/>
+       tibia_length to the farthest point on the tibia body from its joint.
+       coxa_length is the HORIZONTAL-only projection of that real distance
+       (69.49mm), not the full 3D distance (76.41mm) - the real coxa has a
+       small built-in droop too (~25 deg), but the coxa_joint below is pure
+       yaw with zero pitch, so a mesh/kinematics built from the real 3D
+       vector would show the coxa always tilted no matter what q1 is
+       commanded, and every downstream link would inherit a compounding
+       misalignment. Using the horizontal-only length keeps the coxa
+       genuinely level, matching the joint's actual degrees of freedom -
+       the real vertical drop from that droop is what coxa_tilt_deg below
+       absorbs (see its own comment). -->
+  <xacro:property name="coxa_length"  value="0.0695"/>
   <xacro:property name="femur_length" value="0.0859"/>
   <xacro:property name="tibia_length" value="0.1194"/>

Commit message: fix: real hand-measured dimensions, revert to primitive-box rendering
The mesh-alignment work (recent commits) turned into a dead end - real CAD
parts don't sit at the idealized zero-pitch/zero-bend positions the joint
frames assume, and getting per-link mesh origins to actually line up with
the simplified kinematic chain fought every fix. Shelved: use_meshes now
defaults to false again. The mesh files stay in meshes/ in case this gets
revisited, but physics/IK never depended on them anyway (collision is
always the primitive box regardless of use_meshes).

More importantly: the CAD-derived joint coordinates that produced all of
tonight's earlier numbers turned out to imply a ~25 deg coxa droop that
doesn't actually exist on the real hardware - confirmed by Tia directly.
Whatever circles got measured in Fusion weren't the real joint axes.
Replaced with direct hand measurements on the real design:

  coxa_length  0.0695 -> 0.0675 m
  femur_length 0.0859 -> 0.0875 m
  tibia_length 0.1194 -> 0.1075 m (a rubber foot stopper may get added
                                    later - bump this up slightly then)
  body_mount_x 0.1383 -> 0.137865 m
  body_mount_y 0.0663 -> 0.066813 m

coxa_tilt_deg (50 deg) is still the old CAD-derived estimate and is
flagged TODO - still needs a real measurement. leg_splay_deg (40 deg) is
also flagged as a known simplification: the real legs aren't all equally
angled, this assumes symmetric front/rear splay.

Synced hexapod_control/config/gait.yaml and leg_kinematics.py's
LegGeometry defaults per common.xacro's own propagation note. Reach
envelope is now tighter (max femur+tibia reach 195mm vs 205mm before) -
checked existing gait.yaml stride parameters still fit inside it, just
with less margin than before.

Co-Authored-By: Claude Sonnet 5 <noreply@anthropic.com>

File: hexapod_description/urdf/common.xacro (robot description, xacro)
@@ -21,47 +21,43 @@
        tune alongside gait.yaml's stance_drop once the gait is walking. -->
   <xacro:property name="body_height"    value="0.135"/>
-  <!-- Coxa joint positions on the body. Measured from the body-coxa joint's
-       servo-shaft bore in the CAD assembly (see common.xacro's HARDWARE
-       VALUES note - re-measure there first if this changes). -->
-  <xacro:property name="body_mount_x" value="0.1383"/>
-  <xacro:property name="body_mount_y" value="0.0663"/>
+  <!-- Coxa joint positions on the body. Directly measured by Tia on the real
+       design 2026-08-30 (shaft-centre to shaft-centre / body-centre), for
+       the rr leg (x negative, y negative in that leg's own measurement -
+       these properties hold the positive magnitude, hexapod.urdf.xacro
+       applies the sign per leg). -->
+  <xacro:property name="body_mount_x" value="0.137865"/>
+  <xacro:property name="body_mount_y" value="0.066813"/>
   <!-- Leg splay: how far the front/rear legs point off the forward centreline,
        viewed from above. Mid legs are always 90 deg (straight out sideways).
-       Confirmed directly from the body's own mounting-pattern sketch in CAD
-       (measured 140 deg between the forward axis and a rear mount line, i.e.
-       180 - 40). -->
+       NOTE: the real legs are NOT all equally angled from each other -
+       this is a simplified symmetric approximation, not a direct
+       measurement. Revisit with per-leg angles if that asymmetry matters
+       for your gait. -->
   <xacro:property name="leg_splay_deg" value="40"/>
   <!-- ========== leg segments ==========
-       Measured 2026-08-29 from HexapodV2.step: distance between the servo-
-       shaft bore centres at each joint (body-coxa, coxa-femur, femur-tibia),
-       tibia_length to the farthest point on the tibia body from its joint.
-       coxa_length is the HORIZONTAL-only projection of that real distance
-       (69.49mm), not the full 3D distance (76.41mm) - the real coxa has a
-       small built-in droop too (~25 deg), but the coxa_joint below is pure
-       yaw with zero pitch, so a mesh/kinematics built from the real 3D
-       vector would show the coxa always tilted no matter what q1 is
-       commanded, and every downstream link would inherit a compounding
-       misalignment. Using the horizontal-only length keeps the coxa
-       genuinely level, matching the joint's actual degrees of freedom -
-       the real vertical drop from that droop is what coxa_tilt_deg below
-       absorbs (see its own comment). -->
-  <xacro:property name="coxa_length"  value="0.0695"/>
-  <xacro:property name="femur_length" value="0.0859"/>
-  <xacro:property name="tibia_length" value="0.1194"/>
+       Directly measured by Tia on the real design 2026-08-30: shaft-centre
+       to shaft-centre for coxa/femur, shaft-centre to foot tip for tibia.
+       Supersedes the earlier CAD-derived estimates, which turned out to be
+       measuring the wrong reference points (implied a coxa droop that
+       doesn't actually exist on the real hardware). -->
+  <xacro:property name="coxa_length"  value="0.0675"/>
+  <xacro:property name="femur_length" value="0.0875"/>
+  <!-- Tia may add a small rubber foot stopper on top of this later - bump
+       this up slightly if/when that happens. -->
+  <xacro:property name="tibia_length" value="0.1075"/>
   <!-- THE COXA TILT.
        The femur joint's mounting frame is pitched downward relative to the
        coxa, so with all joints at zero the leg already slopes toward the
        ground instead of sticking straight out. This is a fixed mechanical
-       offset in the bracket, NOT a commandable joint. Measured as the real
-       femur droop below horizontal at the CAD's rest pose - the coxa itself
-       also has a smaller built-in droop (~25 deg) that this model doesn't
-       represent separately; folding it into a single tilt at the femur is a
-       deliberate simplification (matches the existing 3-DOF architecture and
-       leg_kinematics.py's planar-arm reduction) rather than adding a second
-       fixed tilt stage.
+       offset in the bracket, NOT a commandable joint. The coxa itself does
+       NOT droop (confirmed 2026-08-30) - all of the leg's fixed tilt lives
+       here, at the femur joint, matching the coxa_joint's actual pure-yaw
+       degrees of freedom.
        Consequence for the IK: the femur command angle is measured FROM this
        tilted frame, so the femur's true angle below horizontal is
        (coxa_tilt_deg + femur_command). hexapod_control accounts for this -
-       see leg_kinematics.py. -->
+       see leg_kinematics.py.
+       TODO: value below is still the old (likely wrong) CAD-derived
+       estimate - needs the real bracket angle. -->
   <xacro:property name="coxa_tilt_deg" value="50"/>
   <xacro:property name="coxa_mass"  value="0.08"/>

File: hexapod_description/urdf/hexapod.urdf.xacro (robot description, xacro)
@@ -14,7 +14,13 @@
        gz_ros2_control plugin can find it at spawn time. -->
   <xacro:arg name="controllers_file" default=""/>
-  <!-- Real meshes landed 2026-08-29 (exported from HexapodV2.step) - on by
-       default now. Set false for the primitive-box fallback. -->
-  <xacro:arg name="use_meshes" default="true"/>
+  <!-- Real mesh files exist in meshes/ (exported from HexapodV2.step,
+       2026-08-29) but getting their per-link origins to actually line up
+       with the simplified kinematic joint frames turned into a real rabbit
+       hole (real CAD parts don't sit at the idealized zero-pitch/zero-bend
+       positions the joints assume) and got shelved. Off by default until
+       that's revisited - the primitive-box fallback below already uses the
+       correct measured dimensions/angles from common.xacro, so physics/IK
+       are unaffected either way; this only changes what it looks like. -->
+  <xacro:arg name="use_meshes" default="false"/>
   <!-- Set false for a plain URDF with no Gazebo / ros2_control tags. -->
   <xacro:arg name="simulation" default="true"/>

Commit message: fix: femur folding into body was two real bugs, not the static geometry
Root-caused by checking actual /joint_states against what was actually
commanded, instead of continuing to guess at the URDF - confirmed the
static geometry (leg.xacro, coxa_tilt_deg, leg_kinematics.py) has been
correct all along (verified three independent ways). Two separate real
bugs were hiding behind what looked like one visual symptom:

1. gait.yaml's neutral stance (stance_reach=80mm, stance_drop=110mm) was
   tuned for older, longer leg dimensions. With the real measured lengths
   (67.5/87.5/107.5mm), reaching that stance target required the femur to
   bend to 106deg below horizontal - past vertical, folding backward
   toward the body instead of continuing outward. New stance_reach=140mm,
   stance_drop=90mm keeps it around 68deg. max_step_length dropped
   0.075->0.030 to stay inside the new (smaller, 195mm) reach envelope at
   this larger stance_reach. body_height (135->90mm) updated to match.

2. Independently, gz_ros2_control's position-holding gain
   (position_proportional_gain) was never actually set, silently running
   on the plugin's default of 0.1 - nowhere near strong enough to track
   position against the new leg mass/geometry under gravity. Confirmed via
   /joint_group_position_controller/commands (correctly commanding 17.9deg
   femur) vs /joint_states (actually sitting at 50.8deg, stable, not just
   still converging) - a real, persistent ~33deg tracking error. Took two
   wrong guesses at the YAML structure (nesting under controller_manager,
   a separate top-level block per joint) before confirming the real
   syntax against gz_ros2_control's own docs: a single global gain under
   its own top-level "gz_ros_control" key, not per-joint. Set to 50.0 -
   verified commanded vs actual now match to within 0.5deg.

Co-Authored-By: Claude Sonnet 5 <noreply@anthropic.com>

File: hexapod_description/urdf/common.xacro (robot description, xacro)
@@ -20,5 +20,5 @@
   <!-- Ride height: ground to base_link origin. Not a direct CAD measurement -
        tune alongside gait.yaml's stance_drop once the gait is walking. -->
-  <xacro:property name="body_height"    value="0.135"/>
+  <xacro:property name="body_height"    value="0.090"/>
   <!-- Coxa joint positions on the body. Directly measured by Tia on the real
        design 2026-08-30 (shaft-centre to shaft-centre / body-centre), for
